File: TPDD_Cable_Z88.sch (KiCad schematic (older format))
At the start: 5 parts, among them J1 Wire Solder Pads, J2 TPDD, Q1 DTA114EKA, Q2 DTA114EKA, Q3 DTA114EKA

Commit message: add WP-2 version, add EB+ in schematics
Connections:
- net EB+: now reaches J2.8 (Pin_8)
Other:
- note added: "Cambridge Z88"
- note added: "External Batt\n+4.8v to +6v"
- note added: "RS-232\n(non-standard pinout)"
- note removed: "RS-232 DTE"
- note removed: "Z88"
Changed lines of the file:
@@
 Text Label 4100 3900 0    50   ~ 0
 CTS_TTL
-Text Notes 7150 3230 0    50   ~ 0
-RS-232 DTE
+Text Notes 6960 3290 0    50   ~ 0
+       RS-232\n(non-standard pinout)
 Wire Wire Line
 	4900 3400 3400 3400
@@
 Wire Wire Line
 	3490 3050 3490 3800
-Text Notes 6780 4750 0    50   ~ 0
+Text Notes 6280 4730 0    50   ~ 0
 DE9M-DE9F extension cable\nCut off female plug.\nSolder wires to J1.\nMatch numbers on pcb silkscreen\nto pin numbers on male connector.
 Wire Wire Line
@@
 Wire Wire Line
 	4500 4000 4500 4400
-Text Notes 7230 3130 0    100  ~ 0
-Z88
+Text Notes 6810 3080 0    100  ~ 0
+Cambridge Z88
 Text Notes 7170 3520 0    50   ~ 0
 DE9 Male
@@
 Text Notes 7270 4240 0    50   ~ 0
 3 RX
+Text Label 4100 4100 0    50   ~ 0
+EB+
+Text Notes 4030 4220 0    30   ~ 0
+External Batt\n+4.8v to +6v
+Wire Notes Line
+	3200 2820 3200 2810
+Wire Notes Line
+	3200 2810 3210 2810
+Wire Notes Line
+	8020 4810 8030 4810
+Wire Notes Line
+	8030 4810 8030 4800
 $EndSCHEMATC
