File: PCB/TPDD_Cable.kicad_pcb (KiCad board)
At the start: 2 copper layers, 10.4 x 13.2 mm, 5 parts, among them J1 Wire Solder Pads, J2 TPDD, Q1 DTA114EKA, Q2 DTA114EKA, Q3 DTA114EKA

Commit message: silkscreen
Routing:
- net /SG: vias 1 -> 4
Other:
- board text added: "${00000000-0000-0000-0000-00005d2d4345:VALUE}"
- board text added: "github bkw777 TPDD_Cable"
- board text added: "v${REVISION}"
- board text removed: "Q* ${00000000-0000-0000-0000-00005d2d4345:VALUE}"
- board text removed: "SIDE"
- board text removed: "THIS"
- board text removed: "tandy.wiki/TPDD"
