File: PCB/TPDD_Cable.kicad_sch (KiCad schematic)
At the start: 5 parts, among them J1 Wire Solder Pads, J2 TPDD, Q1 DTA114EKA, Q2 DTA114EKA, Q3 DTA114EKA

Commit message: pcb version 3
Parts:
- removed J1: Wire Solder Pads, 000_LOCAL:D7_1.5mm_wirepads, symbol 000_LOCAL:1x7_stagger_wirepads
- added P2: RX, 000_LOCAL:PTH_0.65x1.2, symbol 000_LOCAL:TestPoint
- added P20: DSR, 000_LOCAL:PTH_0.65x1.2, symbol 000_LOCAL:TestPoint
- added P3: TX, 000_LOCAL:PTH_0.65x1.2, symbol 000_LOCAL:TestPoint
- added P4: CTS, 000_LOCAL:PTH_0.65x1.2, symbol 000_LOCAL:TestPoint
- added P5: RTS, 000_LOCAL:PTH_0.65x1.2, symbol 000_LOCAL:TestPoint
- added P6: DTR, 000_LOCAL:PTH_0.65x1.2, symbol 000_LOCAL:TestPoint
- added P7: GND, 000_LOCAL:PTH_0.65x1.2, symbol 000_LOCAL:TestPoint
- J2: footprint 000_LOCAL:2-6-2_tpdd -> 000_LOCAL:2x4x2.54mm_edge_mount
Connections:
- net CTS: now also P5.1
- net DSR: now also P4.1
- net DTR: now also P20.1
- net GND: now also P7.1
- net RTS: now also P6.1
- net RX: now also P3.1
- net TX: now also P2.1
Other:
- note added: "(1) Pin 8 TPDD1: N/C TPDD2: External Battery 4.8-6v"
- note added: "DE9F-DB25M Modem cable Cut off DE9F plug. Solder wires, matching numbers on pcb silkscreen to pin numbers on DB25M."
- note removed: "(1) Pin 8 TPDD1: N/C TPDD2: EB+ external battery +4.8v to +6.0v"
- note removed: "DE9F-DB25M Modem cable Cut off DE9F plug. Solder wires to J1. Match numbers on pcb silkscreen to pin numbers on DB25M connector."
- moved on the sheet: J2, Q1, Q2, Q3
