File: PCB/TPDD_Cable_3.kicad_pcb (KiCad board)
At the start: 2 copper layers, 10.4 x 16 mm, 13 parts, among them J2 TPDD, P2 RX, P20 DSR, P3 TX, P4 CTS, P5 RTS, P6 DTR, P7 GND, Q1 DTA114EKA, Q2 DTA114EKA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

Commit message: housing: 0.8mm min-wall & many small fixes. pcb: pull in v1 & v2 pcbs from master & fancy2
Connections:
- net /CTS renamed /TPDD_Cable/CTS
- net /CTS_TTL renamed /TPDD_Cable/CTS_TTL
- net /DSR renamed /TPDD_Cable/DSR
- net /DSR_TTL renamed /TPDD_Cable/DSR_TTL
- net /DTR renamed /TPDD_Cable/DTR
- net /EB+ renamed /TPDD_Cable/EB+
- net /RTS renamed /TPDD_Cable/RTS
- net /RX renamed /TPDD_Cable/RX
- net /RX_TTL renamed /TPDD_Cable/RX_TTL
- net /TX renamed /TPDD_Cable/TX
Other:
- board text added: "github bkw777 TPDD_Cable"
- board text added: "v${REVISION}"
- board text removed: "tandy.wiki"
